File: and-gate.kicad_sch (KiCad schematic)
At the start: 6 parts, among them Q1 NPN, Q2 NPN, Q3 NPN

Commit message: Create PCB layout
Parts:
- removed Q1, Q2, Q3: NPN, symbol Simulation_SPICE:NPN
- added Q13, Q20, Q7: BC547, Package_TO_SOT_THT:TO-92_Inline, symbol Transistor_BJT:BC547
- R5: renamed from R1; footprint (none) -> Resistor_SMD:R_0201_0603Metric
- R6: renamed from R2; footprint (none) -> Resistor_SMD:R_0201_0603Metric
- R7: renamed from R3; footprint (none) -> Resistor_SMD:R_0201_0603Metric
Connections:
- net A: now also Q20.2 (B)
- net B: now also Q13.2 (B)
- net GND: now also Q13.3 (E), Q7.3 (E)
- net OUTPUT: now also Q7.1 (C)
- net at R5.2, R6.1: now also Q20.1 (C)
- net at R6.2: now also Q7.2 (B)
- new net: Q13.1 (C), Q20.3 (E)
