File: control-unit/control-unit.kicad_sch (KiCad schematic)
At the start: 22 parts

Commit message: complete 2-bit encoder
Parts:
- added V1: 5, symbol Simulation_SPICE:VDC
- renumbered ADD to ADD1, CLOCK to CLOCK1, INCREMENT_PC to INCREMENT_PC1, READ_A to READ_A1, READ_B to READ_B1, READ_C to READ_C1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
Connections:
- net INCREMENT_PC: now also INCREMENT_PC1.1 (Pin_1)
- net GND renamed 0
- net 0: now also V1.2
- new net +5V: V1.1
