File: gates/not-gate.kicad_sch (KiCad schematic)
At the start: 3 parts, among them Q20 NPN

Commit message: Use IC circuits in adder circuit
Parts:
- renumbered Q20 to Q12, R25 to R17, R26 to R18
Changed lines of the file:
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@@
 		(dnp no)
 		(fields_autoplaced yes)
-		(property "Reference" "#PWR025"
+		(property "Reference" "#PWR0112"
 			(at 87.63 55.88 0)
 			(effects
@@
 		)
 		(instances
+			(project "register"
+				(path "/176ebc34-d92d-46b0-a9f1-4fb76aa55196/1641c1b9-e3d9-452a-a206-0a4a18cb7a68/6e38e628-9b38-49db-b4e0-13318949e362"
+					(reference "#PWR0112")
+					(unit 1)
+				)
+				(path "/176ebc34-d92d-46b0-a9f1-4fb76aa55196/2b210005-c9ef-43dd-bd20-4304cf65b93c/6e38e628-9b38-49db-b4e0-13318949e362"
+					(reference "#PWR0102")
+					(unit 1)
+				)
+				(path "/176ebc34-d92d-46b0-a9f1-4fb76aa55196/475a755d-c11d-42bc-b5a5-c2bbb617acf6/6e38e628-9b38-49db-b4e0-13318949e362"
+					(reference "#PWR0132")
+					(unit 1)
+				)
+				(path "/176ebc34-d92d-46b0-a9f1-4fb76aa55196/510c109f-9f77-4fcd-9065-7421496291db/6e38e628-9b38-49db-b4e0-13318949e362"
+					(reference "#PWR0122")
+					(unit 1)
+				)
+			)
 			(project "control-unit"
 				(path "/1cf3a7ee-ec47-45b6-b515-1840d726ab8f/020249bf-5e28-4526-a135-e7e504fcd315"
@@
 		(dnp no)
 		(fields_autoplaced yes)
-		(property "Reference" "R25"
+		(property "Reference" "R17"
 			(at 73.66 64.77 90)
 			(effects
@@
 		)
 		(instances
+			(project "register"
+				(path "/176ebc34-d92d-46b0-a9f1-4fb76aa55196/1641c1b9-e3d9-452a-a206-0a4a18cb7a68/6e38e628-9b38-49db-b4e0-13318949e362"
+					(reference "R17")
+					(unit 1)
+				)
+				(path "/176ebc34-d92d-46b0-a9f1-4fb76aa55196/2b210005-c9ef-43dd-bd20-4304cf65b93c/6e38e628-9b38-49db-b4e0-13318949e362"
+					(reference "R1")
+					(unit 1)
+				)
+				(path "/176ebc34-d92d-46b0-a9f1-4fb76aa55196/475a755d-c11d-42bc-b5a5-c2bbb617acf6/6e38e628-9b38-49db-b4e0-13318949e362"
+					(reference "R49")
+					(unit 1)
+				)
+				(path "/176ebc34-d92d-46b0-a9f1-4fb76aa55196/510c109f-9f77-4fcd-9065-7421496291db/6e38e628-9b38-49db-b4e0-13318949e362"
+					(reference "R33")
+					(unit 1)
+				)
+			)
 			(project "control-unit"
 				(path "/1cf3a7ee-ec47-45b6-b515-1840d726ab8f/020249bf-5e28-4526-a135-e7e504fcd315"
@@
 		(dnp no)
 		(fields_autoplaced yes)
-		(property "Reference" "R26"
+		(property "Reference" "R18"
 			(at 90.17 55.8799 0)
 			(effects
@@
 		)
 		(instances
+			(project "register"
+				(path "/176ebc34-d92d-46b0-a9f1-4fb76aa55196/1641c1b9-e3d9-452a-a206-0a4a18cb7a68/6e38e628-9b38-49db-b4e0-13318949e362"
+					(reference "R18")
+					(unit 1)
+				)
+				(path "/176ebc34-d92d-46b0-a9f1-4fb76aa55196/2b210005-c9ef-43dd-bd20-4304cf65b93c/6e38e628-9b38-49db-b4e0-13318949e362"
+					(reference "R2")
+					(unit 1)
+				)
+				(path "/176ebc34-d92d-46b0-a9f1-4fb76aa55196/475a755d-c11d-42bc-b5a5-c2bbb617acf6/6e38e628-9b38-49db-b4e0-13318949e362"
+					(reference "R50")
+					(unit 1)
+				)
+				(path "/176ebc34-d92d-46b0-a9f1-4fb76aa55196/510c109f-9f77-4fcd-9065-7421496291db/6e38e628-9b38-49db-b4e0-13318949e362"
+					(reference "R34")
+					(unit 1)
+				)
+			)
 			(project "control-unit"
 				(path "/1cf3a7ee-ec47-45b6-b515-1840d726ab8f/020249bf-5e28-4526-a135-e7e504fcd315"
@@
 		(dnp no)
 		(fields_autoplaced yes)
-		(property "Reference" "#PWR026"
+		(property "Reference" "#PWR0111"
 			(at 87.63 82.55 0)
 			(effects
@@
 		)
 		(instances
+			(project "register"
+				(path "/176ebc34-d92d-46b0-a9f1-4fb76aa55196/1641c1b9-e3d9-452a-a206-0a4a18cb7a68/6e38e628-9b38-49db-b4e0-13318949e362"
+					(reference "#PWR0111")
+					(unit 1)
+				)
+				(path "/176ebc34-d92d-46b0-a9f1-4fb76aa55196/2b210005-c9ef-43dd-bd20-4304cf65b93c/6e38e628-9b38-49db-b4e0-13318949e362"
+					(reference "#PWR0101")
+					(unit 1)
+				)
+				(path "/176ebc34-d92d-46b0-a9f1-4fb76aa55196/475a755d-c11d-42bc-b5a5-c2bbb617acf6/6e38e628-9b38-49db-b4e0-13318949e362"
+					(reference "#PWR0131")
+					(unit 1)
+				)
+				(path "/176ebc34-d92d-46b0-a9f1-4fb76aa55196/510c109f-9f77-4fcd-9065-7421496291db/6e38e628-9b38-49db-b4e0-13318949e362"
+					(reference "#PWR0121")
+					(unit 1)
+				)
+			)
 			(project "control-unit"
 				(path "/1cf3a7ee-ec47-45b6-b515-1840d726ab8f/020249bf-5e28-4526-a135-e7e504fcd315"
@@
 		(dnp no)
 		(fields_autoplaced yes)
-		(property "Reference" "Q20"
+		(property "Reference" "Q12"
 			(at 90.17 69.8499 0)
 			(effects
@@
 		)
 		(instances
+			(project "register"
+				(path "/176ebc34-d92d-46b0-a9f1-4fb76aa55196/1641c1b9-e3d9-452a-a206-0a4a18cb7a68/6e38e628-9b38-49db-b4e0-13318949e362"
+					(reference "Q12")
+					(unit 1)
+				)
+				(path "/176ebc34-d92d-46b0-a9f1-4fb76aa55196/2b210005-c9ef-43dd-bd20-4304cf65b93c/6e38e628-9b38-49db-b4e0-13318949e362"
+					(reference "Q1")
+					(unit 1)
+				)
+				(path "/176ebc34-d92d-46b0-a9f1-4fb76aa55196/475a755d-c11d-42bc-b5a5-c2bbb617acf6/6e38e628-9b38-49db-b4e0-13318949e362"
+					(reference "Q34")
+					(unit 1)
+				)
+				(path "/176ebc34-d92d-46b0-a9f1-4fb76aa55196/510c109f-9f77-4fcd-9065-7421496291db/6e38e628-9b38-49db-b4e0-13318949e362"
+					(reference "Q23")
+					(unit 1)
+				)
+			)
 			(project "control-unit"
 				(path "/1cf3a7ee-ec47-45b6-b515-1840d726ab8f/020249bf-5e28-4526-a135-e7e504fcd315"
