File: gates/or-gate.kicad_sch (KiCad schematic)
At the start: 7 parts, among them Q1 NPN, Q2 NPN, Q3 NPN

Commit message: Schematic of control-unit
Parts:
- renumbered Q1 to Q7, Q2 to Q8, Q3 to Q9, R5 to R10, R6 to R11, R7 to R12, R4 to R9

Commit message: Assign footprints in half adder
Parts:
- Q1: renamed from Q7; footprint (none) -> SOT-23-3_L2.9-W1.6-P1.90-LS2.8-BR:SOT-23-3_L2.9-W1.6-P1.90-LS2.8-BR
- Q2: renamed from Q8; footprint (none) -> SOT-23-3_L2.9-W1.6-P1.90-LS2.8-BR:SOT-23-3_L2.9-W1.6-P1.90-LS2.8-BR
- Q3: renamed from Q9; footprint (none) -> SOT-23-3_L2.9-W1.6-P1.90-LS2.8-BR:SOT-23-3_L2.9-W1.6-P1.90-LS2.8-BR
- R4: renamed from R9; footprint (none) -> R0603:R0603
- R5: renamed from R10; footprint (none) -> R0603:R0603
- R6: renamed from R11; footprint (none) -> R0603:R0603
- R7: renamed from R12; footprint (none) -> R0603:R0603

Commit message: complete 2-bit encoder
Parts:
- renumbered R4 to R1, R5 to R2, R6 to R3, R7 to R4
Changed lines of the file:
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@@
 		(dnp no)
 		(fields_autoplaced yes)
-		(property "Reference" "#PWR09"
+		(property "Reference" "#PWR05"
 			(at 134.62 78.74 0)
 			(effects
@@
 			(project "control-unit"
 				(path "/1cf3a7ee-ec47-45b6-b515-1840d726ab8f/1729e72d-0a5c-4e1b-b42d-d139718932db"
-					(reference "#PWR09")
+					(reference "#PWR05")
 					(unit 1)
 				)
 				(path "/1cf3a7ee-ec47-45b6-b515-1840d726ab8f/72004cef-785e-4f83-b2f0-4eb1976ff5d3"
-					(reference "#PWR013")
+					(reference "#PWR080")
 					(unit 1)
 				)
 				(path "/1cf3a7ee-ec47-45b6-b515-1840d726ab8f/8e5bfa41-73a7-4155-87a5-165fccd714f6"
-					(reference "#PWR05")
+					(reference "#PWR041")
 					(unit 1)
 				)
@@
 		(dnp no)
 		(fields_autoplaced yes)
-		(property "Reference" "R6"
+		(property "Reference" "R3"
 			(at 137.16 81.2799 0)
 			(effects
@@
 			(project "control-unit"
 				(path "/1cf3a7ee-ec47-45b6-b515-1840d726ab8f/1729e72d-0a5c-4e1b-b42d-d139718932db"
-					(reference "R6")
+					(reference "R3")
 					(unit 1)
 				)
 				(path "/1cf3a7ee-ec47-45b6-b515-1840d726ab8f/72004cef-785e-4f83-b2f0-4eb1976ff5d3"
-					(reference "R15")
+					(reference "R90")
 					(unit 1)
 				)
 				(path "/1cf3a7ee-ec47-45b6-b515-1840d726ab8f/8e5bfa41-73a7-4155-87a5-165fccd714f6"
-					(reference "R11")
+					(reference "R44")
 					(unit 1)
 				)
@@
 		(dnp no)
 		(fields_autoplaced yes)
-		(property "Reference" "#PWR010"
+		(property "Reference" "#PWR06"
 			(at 134.62 143.51 0)
 			(effects
@@
 			(project "control-unit"
 				(path "/1cf3a7ee-ec47-45b6-b515-1840d726ab8f/1729e72d-0a5c-4e1b-b42d-d139718932db"
-					(reference "#PWR010")
+					(reference "#PWR06")
 					(unit 1)
 				)
 				(path "/1cf3a7ee-ec47-45b6-b515-1840d726ab8f/72004cef-785e-4f83-b2f0-4eb1976ff5d3"
-					(reference "#PWR014")
+					(reference "#PWR081")
 					(unit 1)
 				)
 				(path "/1cf3a7ee-ec47-45b6-b515-1840d726ab8f/8e5bfa41-73a7-4155-87a5-165fccd714f6"
-					(reference "#PWR06")
+					(reference "#PWR042")
 					(unit 1)
 				)
@@
 		(dnp no)
 		(fields_autoplaced yes)
-		(property "Reference" "R4"
+		(property "Reference" "R1"
 			(at 111.76 107.95 90)
 			(effects
@@
 			(project "control-unit"
 				(path "/1cf3a7ee-ec47-45b6-b515-1840d726ab8f/1729e72d-0a5c-4e1b-b42d-d139718932db"
-					(reference "R4")
+					(reference "R1")
 					(unit 1)
 				)
 				(path "/1cf3a7ee-ec47-45b6-b515-1840d726ab8f/72004cef-785e-4f83-b2f0-4eb1976ff5d3"
-					(reference "R13")
+					(reference "R88")
 					(unit 1)
 				)
 				(path "/1cf3a7ee-ec47-45b6-b515-1840d726ab8f/8e5bfa41-73a7-4155-87a5-165fccd714f6"
-					(reference "R9")
+					(reference "R42")
 					(unit 1)
 				)
@@
 		(dnp no)
 		(fields_autoplaced yes)
-		(property "Reference" "R5"
+		(property "Reference" "R2"
 			(at 113.03 95.25 90)
 			(effects
@@
 			(project "control-unit"
 				(path "/1cf3a7ee-ec47-45b6-b515-1840d726ab8f/1729e72d-0a5c-4e1b-b42d-d139718932db"
-					(reference "R5")
+					(reference "R2")
 					(unit 1)
 				)
 				(path "/1cf3a7ee-ec47-45b6-b515-1840d726ab8f/72004cef-785e-4f83-b2f0-4eb1976ff5d3"
-					(reference "R14")
+					(reference "R89")
 					(unit 1)
 				)
 				(path "/1cf3a7ee-ec47-45b6-b515-1840d726ab8f/8e5bfa41-73a7-4155-87a5-165fccd714f6"
-					(reference "R10")
+					(reference "R43")
 					(unit 1)
 				)
@@
 		(dnp no)
 		(fields_autoplaced yes)
-		(property "Reference" "#PWR012"
+		(property "Reference" "#PWR08"
 			(at 160.02 119.38 0)
 			(effects
@@
 			(project "control-unit"
 				(path "/1cf3a7ee-ec47-45b6-b515-1840d726ab8f/1729e72d-0a5c-4e1b-b42d-d139718932db"
-					(reference "#PWR012")
+					(reference "#PWR08")
 					(unit 1)
 				)
 				(path "/1cf3a7ee-ec47-45b6-b515-1840d726ab8f/72004cef-785e-4f83-b2f0-4eb1976ff5d3"
-					(reference "#PWR016")
+					(reference "#PWR083")
 					(unit 1)
 				)
 				(path "/1cf3a7ee-ec47-45b6-b515-1840d726ab8f/8e5bfa41-73a7-4155-87a5-165fccd714f6"
-					(reference "#PWR08")
+					(reference "#PWR044")
 					(unit 1)
 				)
@@
 		(dnp no)
 		(fields_autoplaced yes)
-		(property "Reference" "#PWR011"
+		(property "Reference" "#PWR07"
 			(at 160.02 77.47 0)
 			(effects
@@
 			(project "control-unit"
 				(path "/1cf3a7ee-ec47-45b6-b515-1840d726ab8f/1729e72d-0a5c-4e1b-b42d-d139718932db"
-					(reference "#PWR011")
+					(reference "#PWR07")
 					(unit 1)
 				)
 				(path "/1cf3a7ee-ec47-45b6-b515-1840d726ab8f/72004cef-785e-4f83-b2f0-4eb1976ff5d3"
-					(reference "#PWR015")
+					(reference "#PWR082")
 					(unit 1)
 				)
 				(path "/1cf3a7ee-ec47-45b6-b515-1840d726ab8f/8e5bfa41-73a7-4155-87a5-165fccd714f6"
-					(reference "#PWR07")
+					(reference "#PWR043")
 					(unit 1)
 				)
@@
 				)
 				(path "/1cf3a7ee-ec47-45b6-b515-1840d726ab8f/72004cef-785e-4f83-b2f0-4eb1976ff5d3"
-					(reference "Q10")
+					(reference "Q68")
 					(unit 1)
 				)
 				(path "/1cf3a7ee-ec47-45b6-b515-1840d726ab8f/8e5bfa41-73a7-4155-87a5-165fccd714f6"
-					(reference "Q7")
+					(reference "Q31")
 					(unit 1)
 				)
@@
 		(dnp no)
 		(fields_autoplaced yes)
-		(property "Reference" "R7"
+		(property "Reference" "R4"
 			(at 162.56 80.0099 0)
 			(effects
@@
 			(project "control-unit"
 				(path "/1cf3a7ee-ec47-45b6-b515-1840d726ab8f/1729e72d-0a5c-4e1b-b42d-d139718932db"
-					(reference "R7")
+					(reference "R4")
 					(unit 1)
 				)
 				(path "/1cf3a7ee-ec47-45b6-b515-1840d726ab8f/72004cef-785e-4f83-b2f0-4eb1976ff5d3"
-					(reference "R16")
+					(reference "R91")
 					(unit 1)
 				)
 				(path "/1cf3a7ee-ec47-45b6-b515-1840d726ab8f/8e5bfa41-73a7-4155-87a5-165fccd714f6"
-					(reference "R12")
+					(reference "R45")
 					(unit 1)
 				)
@@
 				)
 				(path "/1cf3a7ee-ec47-45b6-b515-1840d726ab8f/72004cef-785e-4f83-b2f0-4eb1976ff5d3"
-					(reference "Q11")
+					(reference "Q69")
 					(unit 1)
 				)
 				(path "/1cf3a7ee-ec47-45b6-b515-1840d726ab8f/8e5bfa41-73a7-4155-87a5-165fccd714f6"
-					(reference "Q8")
+					(reference "Q32")
 					(unit 1)
 				)
@@
 				)
 				(path "/1cf3a7ee-ec47-45b6-b515-1840d726ab8f/72004cef-785e-4f83-b2f0-4eb1976ff5d3"
-					(reference "Q12")
+					(reference "Q70")
 					(unit 1)
 				)
 				(path "/1cf3a7ee-ec47-45b6-b515-1840d726ab8f/8e5bfa41-73a7-4155-87a5-165fccd714f6"
-					(reference "Q9")
-					(unit 1)
-				)
+					(reference "Q33")
+					(unit 1)
+				)

Commit message: Implement logic for jump instruction
Parts:
- renumbered Q1 to Q31, Q2 to Q32, Q3 to Q33, R1 to R42, R2 to R43, R3 to R44, R4 to R45
